File: 555_Timer_Clock.kicad_pcb (KiCad board)
At the start: 2 copper layers, 39 x 25 mm, 13 parts, among them J2 CLK_Out, U1 ICM7555xB

Commit message: 555 Timer Clock Finished Design
Parts:
- added G***: LOGO, LOGO, F.Cu at (105.9, 63.1)
- added J1: +5V, my_footprints:Terminal_Block_5mm, F.Cu at (101.5, 72.4)
- added SW1: Trigger, my_footprints:slide_switch_2.54mm, F.Cu at (122.6, 81.1)
- added SW2: RST, my_footprints:tact_switch_5mm, F.Cu at (112.3, 81.2)
- moved U1 0.28 mm to (124.8, 73.4)
Routing:
- net GND: track 0.00 -> 76.0 mm, vias 0 -> 2
- net /+5V: track 0.00 -> 35.6 mm
- net /Trigger: track 0.00 -> 35.2 mm
- net /CLK_Out: track 0.00 -> 25.1 mm, vias 0 -> 1
- net /RST: track 0.00 -> 17.6 mm
- net Net-(U1-DISCH): track 0.00 -> 13.2 mm
- net Net-(D1-K): track 0.00 -> 9.56 mm
- net Net-(U1-CONT): track 0.00 -> 7.46 mm
